Commit message: 시뮬레이션 차선인식 자동주행 추가 및 맵/속도 스펙 보정
- OpenVINO 차선 모델(models/final_openvino_model)을 온보드 카메라에 연결해
  차선 인식 검증 (sim/lane_detect_preview.py, main.py 파이프라인 오버레이 포함)
- auto.yolo_model, camera fps=30 설정으로 --mode auto 자동 주행 동작 확인
- 도면 스펙(도로폭 850mm) 대비 텍스처 실측으로 맵 크기를 13x9 → 15.085x10.444 m로
  재보정 (k=1.1604, 주차 간격·횡단보도 폭과 교차 검증), 스폰 좌표 동일 배율 적용
- PWM 255 속도를 랩타임 역산으로 0.778 m/s 재보정 → 시뮬레이션 랩타임 47.6초로
  실차 47~48초와 일치 (2랩 검증)
- Prius 시각 메쉬 자산 및 테스트 갱신 (141개 통과)

Co-Authored-By: Claude Fable 5 <noreply@anthropic.com>

File: sim/assets/generated/vehicle.urdf (robot description, URDF)
Before this commit: robot ctrl_zero_child_car, 1 links, 0 joints
Links:
- link rear_axle_frame: geometry visual mesh filename=vehicle_mesh_prius/body.obj; visual mesh filename=vehicle_mesh_prius/glass.obj
